Commit message: chore: clean stale files, update README and media
- Remove legacy hardware drivers and duplicate files from chaska_arm_controller
- Add competition badges and media (sim/real gifs) to README
- Rewrite README: URC/ERC focus, updated PS5 controls, removed roadmap/diagnostics/controllers sections
- Add workspace_status.md to .gitignore
- Camera position adjusted in chaska_arm_base.xacro

File: src/chaska_arm_description/urdf/chaska_arm_base.xacro (robot description, xacro)
@@ -8,6 +8,6 @@
         <mesh filename="package://chaska_arm_description/meshes/base.stl" scale="0.001 0.001 0.001"/>
       </geometry>
-      <material name="pearl_white">
-        <color rgba="0.94 0.94 0.96 1.0"/>
+      <material name="pearl">
+        <color rgba="0.4 0.4 0.4 1.0"/>
       </material>
     </visual>
@@ -33,6 +33,6 @@
         <mesh filename="package://chaska_arm_description/meshes/link_1.stl" scale="0.001 0.001 0.001"/>
       </geometry>
-      <material name="pearl_white">
-        <color rgba="0.94 0.94 0.96 1.0"/>
+      <material name="other_black">
+        <color rgba="0.05 0.05 0.05 1.0"/>
       </material>
     </visual>
@@ -108,6 +108,6 @@
         <mesh filename="package://chaska_arm_description/meshes/link_4.stl" scale="0.001 0.001 0.001"/>
       </geometry>
-      <material name="pearl_white">
-        <color rgba="0.94 0.94 0.96 1.0"/>
+      <material name="other_black">
+        <color rgba="0.05 0.05 0.05 1.0"/>
       </material>
     </visual>
@@ -133,12 +133,12 @@
         <mesh filename="package://chaska_arm_description/meshes/link_5.stl" scale="0.001 0.001 0.001"/>
       </geometry>
-      <material name="pearl_white">
-        <color rgba="0.94 0.94 0.96 1.0"/>
-      </material>
-    </visual>
-    <collision>
-      <origin rpy="0 0 0" xyz="0 0.028 0"/>
-      <geometry>
-        <box size="0.040 0.055 0.040"/>
+      <material name="other_black">
+        <color rgba="0.05 0.05 0.05 1.0"/>
+      </material>
+    </visual>
+    <collision>
+      <origin rpy="0 1.57079632679 0" xyz="0 0 0"/>
+      <geometry>
+        <mesh filename="package://chaska_arm_description/meshes/link_5.stl" scale="0.001 0.001 0.001"/>
       </geometry>
     </collision>
@@ -158,12 +158,12 @@
         <mesh filename="package://chaska_arm_description/meshes/link_6.stl" scale="0.001 0.001 0.001"/>
       </geometry>
-      <material name="pearl_white">
-        <color rgba="0.94 0.94 0.96 1.0"/>
-      </material>
-    </visual>
-    <collision>
-      <origin rpy="0 0 0" xyz="0 0 0"/>
-      <geometry>
-        <box size="0.030 0.060 0.030"/>
+      <material name="other_black">
+        <color rgba="0.05 0.05 0.05 1.0"/>
+      </material>
+    </visual>
+    <collision>
+      <origin rpy="0 1.57079632679 0" xyz="0 0 0"/>
+      <geometry>
+        <mesh filename="package://chaska_arm_description/meshes/link_6.stl" scale="0.001 0.001 0.001"/>
       </geometry>
     </collision>
@@ -288,5 +288,5 @@
     <parent link="link_5"/>
     <child link="depth_camera"/>
-    <origin xyz="0 0.035 0.02" rpy="0 0 1.5708"/>
+    <origin xyz="0 -0.08 0.4" rpy="0 0.6 1.5708"/>
   </joint>
   <joint name="depth_camera_optical_joint" type="fixed">

File: src/rover_description/urdf/rover_base.xacro (robot description, xacro)
@@ -130,6 +130,6 @@
                     <mesh filename="package://rover_description/meshes/yaw.stl" scale="0.001 0.001 0.001"/>
                 </geometry>
-                <material name="black">
-                    <color rgba="0.1 0.1 0.1 1.0"/>
+                <material name="other_black">
+                    <color rgba="0.05 0.05 0.05 1.0"/>
                 </material>
             </visual>
@@ -167,6 +167,6 @@
                     <mesh filename="package://rover_description/meshes/wheel.stl" scale="0.001 0.001 0.001"/>
                 </geometry>
-                <material name="black">
-                    <color rgba="0.1 0.1 0.1 1.0"/>
+                <material name="white">
+                    <color rgba="0.95 0.95 0.95 1.0"/>
                 </material>
             </visual>
@@ -197,6 +197,6 @@
                 <mesh filename="package://rover_description/meshes/base_link.stl" scale="0.001 0.001 0.001"/>
             </geometry>
-            <material name="orange">
-                <color rgba="0.9 0.5 0.1 1.0"/>
+            <material name="other_black">
+                <color rgba="0.05 0.05 0.05 1.0"/>
             </material>
         </visual>
